File: power-board/power-board.kicad_pcb (KiCad board)
At the start: 2 copper layers, 100 x 50 mm, 23 parts, among them J1 LINE/LOAD, J2 DISPLAY, J3 PROG, K1 G3MB-202P, Q1 2N2222A, U1 HLK-PM01, U2 Arduino_pro_mini, U3 MAX6675

Commit message: documentation
Parts:
- removed R7: 100, Resistor_THT:R_Axial_DIN0204_L3.6mm_D1.6mm_P7.62mm_Horizontal
Connections:
- F1 pad 1: Net-(F1-Pad1) -> AC_FUSED
- F1 pad 2: AC_FUSED -> Net-(F1-Pad2)
- F2 pad 2: Net-(F1-Pad1) -> AC_FUSED
- RV1 pad 1: Net-(F1-Pad1) -> AC_FUSED
- U1 pad 1: AC_FUSED -> Net-(F1-Pad2)
- U2 pad 4: Net-(R7-Pad2) -> Net-(BZ1-Pad1)
Routing:
- net Net-(F1-Pad2): track 0.00 -> 19.9 mm
- net Net-(F1-Pad1): track 13.5 -> 0.00 mm
- net Net-(BZ1-Pad1): track 13.9 -> 21.1 mm
- net AC_FUSED: track 19.9 -> 13.5 mm
- net BUTTON_DOWN: track 43.3 -> 37.1 mm
- net Net-(R7-Pad2): track 3.31 -> 0.00 mm
- added copper zone on B.Cu, net AC_FUSED
- removed copper zone on B.Cu, net Net-(F1-Pad1)
